File: libreboard.kicad_pcb (KiCad board)
At the start: 4 copper layers, 125 x 125 mm, 102 parts, among them J100 Screw Terminal, J101 Screw Terminal, J11 USB_C_Receptacle_USB2.0, J12 USB3_A, J13 USB3_A, J14 JST_SHBM04B-SRSS-TB, J15 USB_C_Receptacle_USB2.0, J2 Conn_02x07_Odd_Even, J22 690-019-298-412, J3 Conn_01x03, J4 Bus_M.2_Socket_M, J5 Conn_01x22_Female, J51 12V Fan 1, J52 12V Fan 2, J53 12V Fan 3, J54 12V Fan 4, J7 Micro_SD_Card_Det, J8 THD-20-R, J9 THD-02-R, Q1 CSD18511Q5A, SW1 Right angle Tact button, SW2 Right angle Tact button, U1 TPD4EUSB30, U12 RT9742SNGV, U18 RT9742GGJ5, U2 TPD4EUSB30, U3 MagJack-A70-112-331N126, U4 LM5155DSSR, U5 74LVC1G07SE-7, U6 AP22653W6, U7 ASEK-32.768KHZ-L-R-T, U8 AP3441SHE-7B, U9 SK6812

Commit message: add qwicc
Parts:
- added J16: JST_SHBM04B-SRSS-TB, Connector_JST:JST_SH_BM04B-SRSS-TB_1x04-1MP_P1.00mm_Vertical, F.Cu at (197.2, 148.9)
- H1, H6, H7, H8: footprint MountingHole:MountingHole_3.5mm -> libreboard:MountingHole_2.7mm_M2.5_DIN965
Routing:
- net unconnected-(J16-Pin_2-Pad2): vias 0 -> 1
- net GND: vias 293 -> 292
Other:
- board text added: "Qwiic"
